Commit message: Spawn tribots under unique namespace
All tribots will publish their transforms and topics under unique
namespace. Teleop has namespace as command line argument and control for
each individual tribot twist added.

File: src/tribot_description/urdf/tribot.urdf.xacro (robot description, xacro)
@@ -1,123 +1,112 @@
-<?xml version="1.0" ?>
-<!-- =================================================================================== -->
-<!-- |    This document was autogenerated by xacro from tribot.urdf.xacro              | -->
-<!-- |    EDITING THIS FILE BY HAND IS NOT RECOMMENDED                                 | -->
-<!-- =================================================================================== -->
-<robot name="tribot">
+<?xml version="1.0"?>
+<robot name="tribot" xmlns:xacro="http://ros.org/wiki/xacro">
+  <!-- Define robot constants -->
+  <xacro:property name="base_width" value="0.31" />
+  <xacro:property name="base_length" value="0.42" />
+  <xacro:property name="base_height" value="0.18" />
+  <xacro:property name="wheel_radius" value="0.10" />
+  <xacro:property name="wheel_width" value="0.04" />
+  <xacro:property name="wheel_ygap" value="0.025" />
+  <xacro:property name="wheel_zoff" value="0.05" />
+  <xacro:property name="wheel_xoff" value="0.12" />
+  <xacro:property name="caster_xoff" value="0.14" />
+  <!-- Define intertial property macros  -->
+  <xacro:macro name="box_inertia" params="m w h d">
+    <inertial>
+      <origin xyz="0 0 0" rpy="${pi/2} 0 ${pi/2}" />
+      <mass value="${m}" />
+      <inertia ixx="${(m/12) * (h*h + d*d)}" ixy="0.0" ixz="0.0" iyy="${(m/12) * (w*w + d*d)}" iyz="0.0" izz="${(m/12) * (w*w + h*h)}" />
+    </inertial>
+  </xacro:macro>
+  <xacro:macro name="cylinder_inertia" params="m r h">
+    <inertial>
+      <origin xyz="0 0 0" rpy="${pi/2} 0 0" />
+      <mass value="${m}" />
+      <inertia ixx="${(m/12) * (3*r*r + h*h)}" ixy="0" ixz="0" iyy="${(m/12) * (3*r*r + h*h)}" iyz="0" izz="${(m/2) * (r*r)}" />
+    </inertial>
+  </xacro:macro>
+  <xacro:macro name="sphere_inertia" params="m r">
+    <inertial>
+      <mass value="${m}" />
+      <inertia ixx="${(2/5) * m * (r*r)}" ixy="0.0" ixz="0.0" iyy="${(2/5) * m * (r*r)}" iyz="0.0" izz="${(2/5) * m * (r*r)}" />
+    </inertial>
+  </xacro:macro>
   <!-- Robot Base -->
   <link name="base_link">
     <visual>
       <geometry>
-        <box size="0.42 0.31 0.18"/>
+        <box size="${base_length} ${base_width} ${base_height}" />
       </geometry>
       <material name="Cyan">
-        <color rgba="0 1.0 1.0 1.0"/>
+        <color rgba="0 1.0 1.0 1.0" />
       </material>
     </visual>
     <collision>
       <geometry>
-        <box size="0.42 0.31 0.18"/>
+        <box size="${base_length} ${base_width} ${base_height}" />
       </geometry>
     </collision>
-    <inertial>
-      <origin rpy="1.5707963267948966 0 1.5707963267948966" xyz="0 0 0"/>
-      <mass value="15"/>
-      <inertia ixx="0.261" ixy="0.0" ixz="0.0" iyy="0.34062499999999996" iyz="0.0" izz="0.16062500000000002"/>
-    </inertial>
+    <xacro:box_inertia m="15" w="${base_width}" d="${base_length}" h="${base_height}" />
   </link>
   <!-- Robot Footprint -->
   <link name="base_footprint">
-    <inertial>
-      <origin rpy="1.5707963267948966 0 1.5707963267948966" xyz="0 0 0"/>
-      <mass value="0"/>
-      <inertia ixx="0.0" ixy="0.0" ixz="0.0" iyy="0.0" iyz="0.0" izz="0.0"/>
-    </inertial>
+    <xacro:box_inertia m="0" w="0" d="0" h="0" />
   </link>
   <joint name="base_joint" type="fixed">
-    <parent link="base_link"/>
-    <child link="base_footprint"/>
-    <origin rpy="0 0 0" xyz="0.0 0.0 -0.15000000000000002"/>
-  </joint>
-  <link name="drivewhl_l_link">
+    <parent link="base_link" />
+    <child link="base_footprint" />
+    <origin xyz="0.0 0.0 ${-(wheel_radius+wheel_zoff)}" rpy="0 0 0" />
+  </joint>
+  <!-- Wheels -->
+  <xacro:macro name="wheel" params="prefix x_reflect y_reflect">
+    <link name="${prefix}_link">
+      <visual>
+        <origin xyz="0 0 0" rpy="${pi/2} 0 0" />
+        <geometry>
+          <cylinder radius="${wheel_radius}" length="${wheel_width}" />
+        </geometry>
+        <material name="Gray">
+          <color rgba="0.5 0.5 0.5 1.0" />
+        </material>
+      </visual>
+      <collision>
+        <origin xyz="0 0 0" rpy="${pi/2} 0 0" />
+        <geometry>
+          <cylinder radius="${wheel_radius}" length="${wheel_width}" />
+        </geometry>
+      </collision>
+      <xacro:cylinder_inertia m="0.5" r="${wheel_radius}" h="${wheel_width}" />
+    </link>
+    <joint name="${prefix}_joint" type="continuous">
+      <parent link="base_link" />
+      <child link="${prefix}_link" />
+      <origin xyz="${x_reflect*wheel_xoff} ${y_reflect*(base_width/2+wheel_ygap)} ${-wheel_zoff}" rpy="0 0 0" />
+      <axis xyz="0 1 0" />
+    </joint>
+  </xacro:macro>
+  <xacro:wheel prefix="drivewhl_l" x_reflect="-1" y_reflect="1" />
+  <xacro:wheel prefix="drivewhl_r" x_reflect="-1" y_reflect="-1" />
+  <!-- Caster Wheel -->
+  <link name="front_caster">
     <visual>
-      <origin rpy="1.5707963267948966 0 0" xyz="0 0 0"/>
-      <geometry>
-        <cylinder length="0.04" radius="0.1"/>
-      </geometry>
-      <material name="Gray">
-        <color rgba="0.5 0.5 0.5 1.0"/>
+      <geometry>
+        <sphere radius="${(wheel_radius+wheel_zoff-(base_height/2))}" />
+      </geometry>
+      <material name="Cyan">
+        <color rgba="0 1.0 1.0 1.0" />
       </material>
     </visual>
     <collision>
-      <origin rpy="1.5707963267948966 0 0" xyz="0 0 0"/>
-      <geometry>
-        <cylinder length="0.04" radius="0.1"/>
+      <origin xyz="0 0 0" rpy="0 0 0" />
+      <geometry>
+        <sphere radius="${(wheel_radius+wheel_zoff-(base_height/2))}" />
       </geometry>
     </collision>
-    <inertial>
-      <origin rpy="1.5707963267948966 0 0" xyz="0 0 0"/>
-      <mass value="0.5"/>
-      <inertia ixx="0.0013166666666666667" ixy="0" ixz="0" iyy="0.0013166666666666667" iyz="0" izz="0.0025000000000000005"/>
-    </inertial>
-  </link>
-  <joint name="drivewhl_l_joint" type="continuous">
-    <parent link="base_link"/>
-    <child link="drivewhl_l_link"/>
-    <origin rpy="0 0 0" xyz="-0.12 0.18 -0.05"/>
-    <axis xyz="0 1 0"/>
-  </joint>
-  <link name="drivewhl_r_link">
-    <visual>
-      <origin rpy="1.5707963267948966 0 0" xyz="0 0 0"/>
-      <geometry>
-        <cylinder length="0.04" radius="0.1"/>
-      </geometry>
-      <material name="Gray">
-        <color rgba="0.5 0.5 0.5 1.0"/>
-      </material>
-    </visual>
-    <collision>
-      <origin rpy="1.5707963267948966 0 0" xyz="0 0 0"/>
-      <geometry>
-        <cylinder length="0.04" radius="0.1"/>
-      </geometry>
-    </collision>
-    <inertial>
-      <origin rpy="1.5707963267948966 0 0" xyz="0 0 0"/>
-      <mass value="0.5"/>
-      <inertia ixx="0.0013166666666666667" ixy="0" ixz="0" iyy="0.0013166666666666667" iyz="0" izz="0.0025000000000000005"/>
-    </inertial>
-  </link>
-  <joint name="drivewhl_r_joint" type="continuous">
-    <parent link="base_link"/>
-    <child link="drivewhl_r_link"/>
-    <origin rpy="0 0 0" xyz="-0.12 -0.18 -0.05"/>
-    <axis xyz="0 1 0"/>
-  </joint>
-  <!-- Caster Wheel -->
-  <link name="front_caster">
-    <visual>
-      <geometry>
-        <sphere radius="0.060000000000000026"/>
-      </geometry>
-      <material name="Cyan">
-        <color rgba="0 1.0 1.0 1.0"/>
-      </material>
-    </visual>
-    <collision>
-      <origin rpy="0 0 0" xyz="0 0 0"/>
-      <geometry>
-        <sphere radius="0.060000000000000026"/>
-      </geometry>
-    </collision>
-    <inertial>
-      <mass value="0.5"/>
-      <inertia ixx="0.0007200000000000006" ixy="0.0" ixz="0.0" iyy="0.0007200000000000006" iyz="0.0" izz="0.0007200000000000006"/>
-    </inertial>
+    <xacro:sphere_inertia m="0.5" r="${(wheel_radius+wheel_zoff-(base_height/2))}" />
   </link>
   <joint name="caster_joint" type="fixed">
-    <parent link="base_link"/>
-    <child link="front_caster"/>
-    <origin rpy="0 0 0" xyz="0.14 0.0 -0.09"/>
+    <parent link="base_link" />
+    <child link="front_caster" />
+    <origin xyz="${caster_xoff} 0.0 ${-(base_height/2)}" rpy="0 0 0" />
   </joint>
   <!-- Imu Sensor-->
@@ -125,22 +114,18 @@
     <visual>
       <geometry>
-        <box size="0.1 0.1 0.1"/>
+        <box size="0.1 0.1 0.1" />
       </geometry>
     </visual>
     <collision>
       <geometry>
-        <box size="0.1 0.1 0.1"/>
+        <box size="0.1 0.1 0.1" />
       </geometry>
     </collision>
-    <inertial>
-      <origin rpy="1.5707963267948966 0 1.5707963267948966" xyz="0 0 0"/>
-      <mass value="0.1"/>
-      <inertia ixx="0.0001666666666666667" ixy="0.0" ixz="0.0" iyy="0.0001666666666666667" iyz="0.0" izz="0.0001666666666666667"/>
-    </inertial>
+    <xacro:box_inertia m="0.1" w="0.1" d="0.1" h="0.1" />
   </link>
   <joint name="imu_joint" type="fixed">
-    <parent link="base_link"/>
-    <child link="imu_link"/>
-    <origin xyz="0 0 0.01"/>
+    <parent link="base_link" />
+    <child link="imu_link" />
+    <origin xyz="0 0 0.01" />
   </joint>
   <gazebo reference="imu_link">
@@ -215,24 +200,24 @@
   <link name="laser_link">
     <visual>
-      <origin rpy="0 0 0" xyz="0 0 0"/>
-      <geometry>
-        <cylinder length="0.1" radius="0.05"/>
-      </geometry>
-      <material name="white"/>
+      <origin xyz="0 0 0" rpy="0 0 0" />
+      <geometry>
+        <cylinder radius="0.05" length="0.1"/>
+      </geometry>
+      <material name="white" />
     </visual>
     <collision>
-      <origin rpy="0 0 0" xyz="0 0 0"/>
-      <geometry>
-        <cylinder length="0.1" radius="0.05"/>
+      <origin xyz="0 0 0" rpy="0 0 0"/>
+      <geometry>
+        <cylinder radius="0.05" length="0.1"/>
       </geometry>
     </collision>
   </link>
   <joint name="joint_sensor_laser" type="fixed">
-    <origin rpy="0 0 0" xyz="0.15 0 0.05"/>
+    <origin xyz="0.15 0 0.05" rpy="0 0 0"/>
     <parent link="base_link"/>
     <child link="laser_link"/>
   </joint>
   <gazebo reference="sensor_laser">
-    <sensor name="head_hokuyo_sensor" type="ray">
+    <sensor type="ray" name="head_hokuyo_sensor">
       <pose>0 0 0 0 0 0</pose>
       <visualize>false</visualize>
@@ -258,5 +243,5 @@
         </noise>
       </ray>
-      <plugin filename="libgazebo_ros_laser.so" name="gazebo_ros_head_hokuyo_controller">
+      <plugin name="gazebo_ros_head_hokuyo_controller" filename="libgazebo_ros_laser.so">
         <topicName>/m2wr/laser/scan</topicName>
         <frameName>sensor_laser</frameName>
@@ -266,5 +251,5 @@
   <!--Differential drive plugin-->
   <gazebo>
-    <plugin filename="libgazebo_ros_diff_drive.so" name="diff_drive_plugin">
+    <plugin name='diff_drive_plugin' filename='libgazebo_ros_diff_drive.so'>
       <ros>
         <!--namespace>/demo</namespace-->
@@ -290,19 +275,19 @@
   <link name="battery_link">
     <inertial>
-      <inertia ixx="0.00001" ixy="0.0" ixz="0.0" iyy="0.00001" iyz="0.0" izz="0.00001"/>
-      &gt;
-      <mass value="0.001"/>
-      <origin rpy="0 0 0" xyz="0 0 0"/>
+      <inertia ixx="0.00001" ixy="0.0" ixz="0.0" iyy="0.00001" iyz="0.0" izz="0.00001" />>
+      <mass value="0.001" />
+      <origin xyz="0 0 0" rpy="0 0 0" />
     </inertial>
   </link>
   <joint name="battery_joint" type="revolute">
-    <origin rpy="0 0 0" xyz="0 0 0"/>
+    <origin xyz="0 0 0" rpy="0 0 0"/>
     <parent link="base_link"/>
     <child link="battery_link"/>
     <axis xyz="1 0 0"/>
-    <limit effort="0" lower="0" upper="0" velocity="0"/>
+    <limit upper="0" lower="0" effort="0" velocity="0"/>
   </joint>
   <gazebo>
-    <plugin filename="libgazebo_ros_linear_battery.so" name="linear_battery_plugin">
+    <plugin filename="libgazebo_ros_linear_battery.so"
+    name="linear_battery_plugin">
       <ros>
         <!--namespace>/demo</namespace-->
